File: cho-corne-ice/pcb/cho-corne-ice-Both.kicad_pcb (KiCad board)
At the start: 2 copper layers, 275.5 x 105.6 mm, 120 parts, among them J1 BAT, J2 nice!view, J3 BAT, J4 nice!view, SW1 SW_PUSH, SW10 SW_PUSH, SW11 SW_PUSH, SW12 SW_PUSH, SW13 SW_PUSH, SW14 SW_PUSH, SW15 SW_PUSH, SW16 SW_PUSH, SW17 SW_PUSH, SW18 SW_PUSH, SW19 SW_PUSH, SW2 SW_PUSH, SW20 SW_PUSH, SW21 SW_PUSH, SW22 SW_PUSH, SW23 SW_PUSH, SW24 SW_PUSH, SW25 SW_PUSH, SW26 SW_PUSH, SW27 SW_PUSH, SW28 SW_PUSH, SW29 SW_PUSH, SW3 SW_PUSH, SW30 SW_PUSH, SW31 SW_PUSH, SW32 SW_PUSH, SW33 SW_PUSH, SW34 SW_PUSH, SW35 SW_PUSH, SW36 SW_PUSH, SW37 SW_PUSH, SW38 SW_PUSH, SW39 SW_PUSH, SW4 SW_PUSH, SW40 SW_PUSH, SW41 SW_PUSH, SW42 SW_PUSH, SW5 SW_PUSH, SW6 SW_PUSH, SW7 SW_PUSH, SW8 SW_PUSH, SW9 SW_PUSH, U1 nice!nano, U2 nice!nano

Commit message: split left and right into own pcb files
Parts:
- removed REF** (x8): Breakaway_Tabs, kbd:Breakaway_Tabs
Other:
- board size 275.5 x 105.6 mm -> 274.5 x 91.4 mm
- board text added: "Cho-Corne-Ice v0.2 PCB Designed by foostan/e3b0c442/badjeff"
- board text removed: "Cho-Corne-Ice v0.2 PCB Designed by foostan/e3b0c442"
